File: Hardware/JumperlessV5hw/JustTheLEDs.kicad_sch (KiCad schematic)
At the start: 446 parts

Commit message: Changed caps on rail power supplies
Parts:
- removed D1, D10, D11, D12, D13, D14, D15, D16, D17, D18, D19, D2, D20, D21, D22, D23, D24, D25, D26, D27, D28, D29, D3, D30, D31, D32, D33, D4, D5, D6, D7, D8, D9: WS2812B, LED_SMD:LED_SK6812_EC15_1.5x1.5mm, symbol JumperlessSymbols:xl-1010RGBC
Other:
- moved on the sheet: C28, C29, C30, C31, C32, C33, C34, C35, C36, C37, D1011, D1012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

Commit message: Rearranged the schematic for prettyness
Other:
- company: (none) -> Architeuthis Flux
- title: (none) -> Jumperless V5
Changed lines of the file:
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@@
 	(generator_version "8.0")
 	(paper "A0")
+	(title_block
+		(title "Jumperless V5")
+		(date "2024-06-15")
+		(rev "5r2")
+		(company "Architeuthis Flux")
+		(comment 1 "Kevin Santo Cappuccio")
+		(comment 2 "KevinC@ppucc.io")
+	)
 	(junction
 		(at 194.31 486.41)
