File: Hardware/JumperlessV5hw/JumperlessV5hw.kicad_sch (KiCad schematic)
At the start: 183 parts, among them J1 Debug, J11 TopOutMAIN, J12 TopInMAIN, J13 BottomInMAIN, J14 5V, J15 BottomOutMAIN, J1711 Conn_01x15, J1712 Conn_01x15, J2 USB_C_Receptacle_USB2.0_16P, J3 ProbeJack, J4 Breadboard, J5 ProbeHeader, J6 CH446Q, J7 DaisyChain_OUT, J8 DaisyChain_IN, K1 CH446Q, SW1 BOOT, SW3 RotaryEncoder_Switch, U1 LT1054, U10 L272D, U11 LM324, U1806 MCP4728, U1807 L272D, U1808 MCP23S17_ML, U2 NCP1117-3.3_SOT223, U3 INA219, U4 INA219, U7 LM324, U8 W25Q128JVS, U9 RP2040, Y1 ABLS-12.000MHZ-B4-T

Commit message: Changed caps on rail power supplies
Parts:
- C1806, C1807: value 10uF -> 0.1uF
Changed lines of the file:
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@@
 		)
 	)
-	(global_label "GPIO_7"
-		(shape bidirectional)
-		(at 322.58 261.62 180)
-		(fields_autoplaced yes)
-		(effects
-			(font
-				(size 1.27 1.27)
-			)
-			(justify right)
-		)
-		(property "Intersheetrefs" "${INTERSHEET_REFS}"
-			(at 311.8311 261.62 0)
-			(effects
-				(font
-					(size 1.27 1.27)
-				)
-				(justify right)
-				(hide yes)
-			)
-		)
-	)
 	(global_label "GPIO_22"
 		(shape bidirectional)
@@
 		)
 	)
-	(global_label "GPIO_2"
-		(shape bidirectional)
-		(at 322.58 244.475 180)
-		(fields_autoplaced yes)
-		(effects
-			(font
-				(size 1.27 1.27)
-			)
-			(justify right)
-		)
-		(property "Intersheetrefs" "${INTERSHEET_REFS}"
-			(at 311.8311 244.475 0)
-			(effects
-				(font
-					(size 1.27 1.27)
-				)
-				(justify right)
-				(hide yes)
-			)
-		)
-	)
 	(global_label "DL"
 		(shape bidirectional)
@@
 		)
 	)
-	(global_label "GPIO_6"
-		(shape bidirectional)
-		(at 322.58 256.54 180)
-		(fields_autoplaced yes)
-		(effects
-			(font
-				(size 1.27 1.27)
-			)
-			(justify right)
-		)
-		(property "Intersheetrefs" "${INTERSHEET_REFS}"
-			(at 311.8311 256.54 0)
-			(effects
-				(font
-					(size 1.27 1.27)
-				)
-				(justify right)
-				(hide yes)
-			)
-		)
-	)
 	(global_label "44"
 		(shape bidirectional)
@@
 		)
 	)
-	(global_label "GPIO_3"
-		(shape bidirectional)
-		(at 322.58 250.19 180)
-		(fields_autoplaced yes)
-		(effects
-			(font
-				(size 1.27 1.27)
-			)
-			(justify right)
-		)
-		(property "Intersheetrefs" "${INTERSHEET_REFS}"
-			(at 311.8311 250.19 0)
-			(effects
-				(font
-					(size 1.27 1.27)
-				)
-				(justify right)
-				(hide yes)
-			)
-		)
-	)
 	(global_label "CS_I"
 		(shape input)
@@
 			)
 		)
-		(property "Value" "10uF"
+		(property "Value" "0.1uF"
 			(at 776.351 274.828 0)
 			(effects
@@
 			)
 		)
-		(property "Value" "10uF"
+		(property "Value" "0.1uF"
 			(at 781.431 321.818 0)
 			(effects
@@
 	(symbol
 		(lib_id "Device:R_Pack04_Split")
-		(at 827.405 346.075 0)
+		(at 871.855 346.71 0)
 		(unit 3)
 		(exclude_from_sim no)
@@
 		(dnp no)
 		(property "Reference" "RN9"
-			(at 827.405 348.615 90)
+			(at 871.855 349.25 90)
 			(effects
 				(font
@@
 		)
 		(property "Value" "47K"
-			(at 827.405 347.98 90)
+			(at 871.855 348.615 90)
 			(effects
 				(font
@@
 		)
 		(property "Footprint" "Resistor_SMD:R_Array_Convex_4x0402"
-			(at 825.373 346.075 90)
+			(at 869.823 346.71 90)
 			(effects
 				(font
@@
 		)
 		(property "Datasheet" "~"
-			(at 827.405 346.075 0)
+			(at 871.855 346.71 0)
 			(effects
 				(font
@@
 		)
 		(property "Description" "4 resistor network, parallel topology, split"
-			(at 827.405 346.075 0)
+			(at 871.855 346.71 0)
 			(effects
 				(font
@@
 		)
 		(property "LCSC" " C2769517"
-			(at 827.405 346.075 90)
+			(at 871.855 346.71 90)
 			(effects
 				(font
@@
 		)
 		(property "LCSC Part #" " C2769517"
-			(at 827.405 346.075 0)
+			(at 871.855 346.71 0)
 			(effects
 				(font
@@
 	(symbol
 		(lib_id "Device:R_Pack04_Split")
-		(at 831.85 319.405 90)
+		(at 876.3 320.04 90)
 		(unit 3)
 		(exclude_from_sim no)
@@
 		(dnp no)
 		(property "Reference" "RN11"
-			(at 834.39 319.405 90)
+			(at 878.84 320.04 90)
 			(effects
 				(font
@@
 		)
 		(property "Value" "56K"
-			(at 833.755 319.405 90)
+			(at 878.205 320.04 90)
 			(effects
 				(font
@@
 		)
 		(property "Footprint" "Resistor_SMD:R_Array_Convex_4x0402"
-			(at 831.85 321.437 90)
+			(at 876.3 322.072 90)
 			(effects
 				(font
@@
 		)
 		(property "Datasheet" "+-1%"
-			(at 831.85 319.405 0)
+			(at 876.3 320.04 0)
 			(effects
 				(font
@@
 		)
 		(property "Description" "4 resistor network, parallel topology, split "
-			(at 831.85 319.405 0)
+			(at 876.3 320.04 0)
 			(effects
 				(font
@@
 		)
 		(property "LCSC" " C425288"
-			(at 831.85 319.405 90)
+			(at 876.3 320.04 90)
 			(effects
 				(font
@@
 		)
 		(property "LCSC Part #" " C425288"
-			(at 831.85 319.405 0)
+			(at 876.3 320.04 0)
 			(effects
 				(font
@@
 	(symbol
 		(lib_id "Device:R_Pack04_Split")
-		(at 815.34 324.485 0)
+		(at 859.79 325.12 0)
 		(unit 4)
 		(exclude_from_sim no)
@@
 		(dnp no)
 		(property "Reference" "RN11"
-			(at 815.34 327.025 90)
+			(at 859.79 327.66 90)
 			(effects
 				(font
@@
 		)
 		(property "Value" "56K"
-			(at 815.34 326.39 90)
+			(at 859.79 327.025 90)
 			(effects
 				(font
@@
 		)
 		(property "Footprint" "Resistor_SMD:R_Array_Convex_4x0402"
-			(at 813.308 324.485 90)
+			(at 857.758 325.12 90)
 			(effects
 				(font
@@
 		)
 		(property "Datasheet" "+-1%"
-			(at 815.34 324.485 0)
+			(at 859.79 325.12 0)
 			(effects
 				(font
@@
 		)
 		(property "Description" "4 resistor network, parallel topology, split "
-			(at 815.34 324.485 0)
+			(at 859.79 325.12 0)
 			(effects
 				(font
@@
 		)
 		(property "LCSC" " C425288"
-			(at 815.34 324.485 90)
+			(at 859.79 325.12 90)
 			(effects
 				(font
@@
 		)
 		(property "LCSC Part #" " C425288"
-			(at 815.34 324.485 0)
+			(at 859.79 325.12 0)
 			(effects
 				(font

Commit message: Rearranged the schematic for prettyness
Parts:
- removed unit 3 of RN11
- removed unit 4 of RN11
- removed unit 3 of RN9
- RN1, RN2, RN3: now not fitted
Other:
- note added: "All the LEDs are down here"
- note added: "Daisy Chain Headers"
- note added: "Do Not Place these pulldowns"
- note added: "Don't worry about this crap"
- note added: "GPIO Expander"
- note added: "I2C Pullups"
- note added: "Probe Connectors"
- note added: "Probe Sense Pads"
- note added: "Rotary Encoder"
- note removed: "Added in Rev 3"
- note removed: "Power Cutoff for power Op Amp"
- company: (none) -> Architeuthis Flux
- title: (none) -> Jumperless V5
- moved on the sheet: A1, A2, B1, C1, C10, C11, C12, C13, C14, C15, C16, C17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

Commit message: Getting probing to work and a bunch of other stuff
Other:
- note added: "Change this to GPIO or something +-8V tolerant ----------->"
Changed lines of the file:
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@@
+		)
+	)
+	(text "Change this to GPIO\nor something +-8V \ntolerant ----------->"
+		(exclude_from_sim no)
+		(at 653.034 128.524 0)
+		(effects
+			(font
+				(size 1.27 1.27)
+			)
+			(justify left)
 		)
 	)

Commit message: Hackin' away at shit
Parts:
- removed RN1, RN2, RN3: 10K, Resistor_SMD:R_Array_Convex_4x0402, symbol Device:R_Pack04_Split
- removed unit 3 of RN10
- removed unit 4 of RN10
- removed unit 4 of RN8
- removed unit 3 of RN8
- added RN11: 1M, Resistor_SMD:R_Array_Convex_4x0402, symbol Device:R_Pack04_Split
- added TP15: LED IN_FROM_WISHBONE, JumperlessFootprints:PINHEADER-1x1_vertical, symbol JumperlessSymbols:TestPoint
- C2, C3, C5: footprint Capacitor_Tantalum_SMD:CP_EIA-6032-20_AVX-F_Pad2.25x2.35mm_HandSolder -> Capacitor_Tantalum_SMD:CP_EIA-3528-12_Kemet-T_Pad1.50x2.35mm_HandSolder
- R21, R55, R56, R58, R59, R60, R61, R62, R63, R64, R65, R66, R67, R68, R69, R70, R71, R72, R73, R74, R75, R76, R77, R78: value 47 -> 22; LCSC C137973 -> C114765; LCSC Part # C137973 -> C114765
- RN10: LCSC C425288 -> C621323; LCSC Part # C425288 -> C621323
- RN10: renamed from RN11; LCSC C425288 -> C621323; LCSC Part # C425288 -> C621323
- TP7: value 0-5V DAC -> DAC_0
- TP8: value +-8V DAC -> DAC_1
Connections:
- net +5V: now also U1807.4 (V+)
- net +9V: no longer U1807.4 (V+)
- net -9V: no longer U1807.6 (V-)
- net ADC_UNBUFFERED_+-8V_2: now also RN11.6 (R3.2)
- net ADC_UNBUFFERED_+-8V_3: now also RN11.5 (R4.2)
- net ADC_UNBUFFERED_5V_1: now also RN11.7 (R2.2)
- net BOTTOM_RAIL: now also U1807.11 (-)
- net GND: now also J3.3 (R1), RN10.3 (R3.1), U1807.6 (V-), RN11.1 (R1.1), RN11.2 (R2.1), RN11.3 (R3.1), RN11.4 (R4.1); no longer RN10.2 (R2.1)
- net I2C_SCL: no longer J3.5 (R3)
- net I2C_SDA: no longer J3.4 (R2)
- net Probe_Button: now also J3.5 (R3); no longer J3.1 (S)
- net ROUTABLE_BUFFER_IN: now also J3.1 (S), RN11.8 (R1.2); no longer J3.3 (R1)
- net R_SENSE+: now also RN8.2 (R2.1); no longer U10.14 (-)
- net TOP_RAIL: now also U1807.14 (-); no longer RN8.2 (R2.1)
- net at RN9.2 (R2.1): now also RN10.4 (R4.1); no longer RN10.1 (R1.1)
- net at RN10.8 (R1.2), RN12.8 (R1.2): now also U10.14 (-); no longer U1807.14 (-)
- net at RN12.2 (R2.1): no longer U1807.11 (-)
- net at RN12.5 (R4.2), RN9.1 (R1.1): now also RN10.6 (R3.2); no longer RN10.7 (R2.2)
- net at RN12.4 (R4.1), U10.11 (-): now also RN10.5 (R4.2); no longer RN10.8 (R1.2)
- net DAC_+-8V renamed DAC_1
- net DAC_0-5V renamed DAC_0
- new net LED_446: J3.4 (R2), TP15.1
Other:
- note added: "Make these 0-5V"
- note removed: "Change this to GPIO or something +-8V tolerant ----------->"
- note removed: "Do Not Place these pulldowns"
- moved on the sheet: A1, A2, B1, C1, C10, C11, C12, C13, C14, C15, C16, C17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

Commit message: Now with RP2350B!
Parts:
- removed C16, C25: 10uF, Capacitor_SMD:C_0603_1608Metric, symbol JumperlessSymbols:C_Small
- added JP3: Rail Cutoff Top, JumperlessFootprints:SolderJumper_2_Bridged_Small, symbol JumperlessSymbols:SolderJumper_2_Bridged
- added JP4: Rail Cutoff Bottom, JumperlessFootprints:SolderJumper_2_Bridged_Small, symbol JumperlessSymbols:SolderJumper_2_Bridged
- added Q3: Q_NPN_CBE, symbol Device:Q_NPN_CBE
- added R6: 1K, Resistor_SMD:R_0402_1005Metric_Pad0.72x0.64mm_HandSolder, symbol Device:R_Small_US
- added R7: 0R, Resistor_SMD:R_0402_1005Metric_Pad0.72x0.64mm_HandSolder, symbol Device:R_Small_US
- added TP2: TestPoint, JumperlessFootprints:TestPoint_Pad_D1.0mm, symbol Connector:TestPoint
- C1806, C1807: value 0.1uF -> 1uF
- C2, C3, C5: LCSC C139814 -> C189401
- R21, R55, R56, R58, R59, R60, R61, R62, R63, R64, R65, R66, R67, R68, R69, R70, R71, R72, R73, R74, R75, R76, R77, R78: value 22 -> 33
Connections:
- net BOTTOM_RAIL: now also JP4.2 (B); no longer C1807.1, U1807.11 (-), U1807.5
- net GND: now also J3.1 (S), R6.2; no longer J3.3 (R1)
- net GPIO_2: now also J3.4 (R2)
- net LED_446: now also TP2.1; no longer J3.4 (R2)
- net Probe_Button: now also J3.3 (R1); no longer J3.5 (R3)
- net ROUTABLE_BUFFER_IN: now also J3.5 (R3); no longer J3.1 (S)
- net TOP_RAIL: now also JP3.2 (B); no longer C1806.1, U1807.14 (-), U1807.3
- net at C4.2, U1.5 (-VOUT): now also Q3.3 (E), R7.1; no longer D65.1 (K)
- new net: C1806.1, JP3.1 (A), U1807.14 (-), U1807.3
- new net: C1807.1, JP4.1 (A), U1807.11 (-), U1807.5
- new net: D65.1 (K), Q3.1 (C), R7.2
- new net: Q3.2 (B), R6.1
Other:
- note added: "We're gonna use TRRS cables, so GPIO 2 and Button are shorted"
- moved on the sheet: C1806, C1807, C4, RN4A, RN4B, RN4C, RN4D, TP6, U1807A, U1807B, U1807C
