File: Hardware/Jumperless23V50/JustTheLEDs.kicad_sch (KiCad schematic)
At the start: 413 parts

Commit message: Add FPC breakout and almost finished V5r4
Connections:
- net LED_60_OUT: now reaches D1605.1 (DOUT)
- net LED_60_OUT: no longer D1611.4 (DIN)
- new net LED_RAILS_IN: D1611.4 (DIN)
Changed lines of the file:
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@@
 	(wire
 		(pts
-			(xy 1158.24 326.39) (xy 63.5 326.39)
-		)
-		(stroke
-			(width 0)
-			(type default)
-		)
-	)
-	(wire
-		(pts
 			(xy 245.11 400.05) (xy 245.11 415.29)
 		)
@@
 				(hide yes)
 			)
+		)
+	)
+	(global_label "LED_60_OUT"
+		(shape output)
+		(at 1158.24 326.39 0)
+		(fields_autoplaced yes)
+		(effects
+			(font
+				(size 1.27 1.27)
+			)
+			(justify left)
+		)
+		(property "Intersheetrefs" "${INTERSHEET_REFS}"
+			(at 1172.6551 326.39 0)
+			(effects
+				(font
+					(size 1.27 1.27)
+				)
+				(justify left)
+				(hide yes)
+			)
+		)
+	)
+	(global_label "LED_RAILS_IN"
+		(shape input)
+		(at 63.5 326.39 0)
+		(fields_autoplaced yes)
+		(effects
+			(font
+				(size 1.27 1.27)
+			)
+			(justify left)
+		)
+		(property "Intersheetrefs" "${INTERSHEET_REFS}"
+			(at 79.0038 326.39 0)
+			(effects
+				(font
+					(size 1.27 1.27)
+				)
+				(justify left)
+				(hide yes)
+			)
