File: Jumperless23V50/JumperlessV5r6/JumperlessV5r6/JumperlessV5r6.kicad_sch (KiCad schematic)
At the start: 235 parts, among them J1 Debug, J11 TopOutMAIN, J12 TopInMAIN, J13 BottomInMAIN, J14 5V, J15 BottomOutMAIN, J1711 Conn_01x15, J1712 Conn_01x15, J2 USB_C_Receptacle_USB2.0_16P, J3 ProbeJack, J4 Breadboard, J5 FPC Connector, J6 CH446Q, J7 DaisyChain_OUT, J8 DaisyChain_IN, K1 CH446Q, SW1 BOOT, SW3 RotaryEncoder_Switch, U1 LT1054, U10 L272D, U11 LM324, U1806 MCP4728, U1807 L272D, U2 NCP1117-3.3_SOT223, U3 INA219, U4 INA219, U5 RP2350_80QFN, U6 TLV73311PDBV, U7 LM324, U8 W25Q128JVS, U9 LM2660MX, Y1 ABM8-272-T3

Commit message: made a schematic with everything on one sheet
Other:
- moved on the sheet: R21, R55, R56, R58, R59, R60, R61, R62, R63, R64, R65, R66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
