File: Jumperless23V50/JumperlessV5r6/JumperlessV5r6/JustTheLEDs.kicad_sch (KiCad schematic)
At the start: 413 parts

Commit message: made a schematic with everything on one sheet
Other:
- note added: "1 2 3 4 5 6 7 8 9 10 11 12 13 14 15 16 17 18 19 20 21 22 23 24 25 26 27 28 29 30"
- note added: "31 32 33 34 35 36 37 38 39 40 41 42 43 44 45 46 47 48 49 50 51 52 53 54 55 56 57 58 59 60"
- moved on the sheet: C28, C29, C30, C31, C32, C33, C34, C35, C36, C37, D1611, D1612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
