File: Jumperless23V50/V5probe/V5probe.kicad_sch (KiCad schematic)
At the start: 44 parts, among them J1 Conn_01x05_Socket, J2 Probe Needle, J7 ProbeJack, SW1 Disconnect, SW3 Connect, SW4 SW_DPDT_x2, U1 WS2811

Commit message: Work with Wokwi's new backend
Parts:
- removed TP9: Din, JumperlessFootprints:TestPoint_D0.75mm, symbol JumperlessSymbols:TestPoint
Other:
- note added: "Connect Disconnect Measure"
- note removed: "Measure Disconnect Connect"
- note removed: "We're gonna use TRRS cables, so LED_OUT_PROBE and Button are shorted"
- moved on the sheet: C1, D1, D5, J7, JP1, JP3, JP4, JP5, JP6, JP7, JP9, R3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
