File: Jumperless23V50/MainBoard/JumperlessV5r6/JumperlessV5r6.kicad_sch (KiCad schematic)
At the start: 235 parts, among them J1 Debug, J11 TopOutMAIN, J12 TopInMAIN, J13 BottomInMAIN, J14 5V, J15 BottomOutMAIN, J1711 Conn_01x15, J1712 Conn_01x15, J2 USB_C_Receptacle_USB2.0_16P, J3 ProbeJack, J4 Breadboard, J5 FPC Connector, J6 CH446Q, J7 DaisyChain_OUT, J8 DaisyChain_IN, K1 CH446Q, SW1 BOOT, SW3 RotaryEncoder_Switch, U1 LT1054, U10 L272D, U11 LM324, U1806 MCP4728, U1807 L272D, U2 NCP1117-3.3_SOT223, U3 INA219, U4 INA219, U5 RP2350_80QFN, U6 TLV73311PDBV, U7 LM324, U8 W25Q128JVS, U9 LM2660MX, Y1 ABM8-272-T3

Commit message: Add related repos as submodules, rev7 hardware update
Parts:
- removed R89: 0R, Resistor_SMD:R_0402_1005Metric_Pad0.72x0.64mm_HandSolder, symbol Device:R_Small_US
- removed U6: TLV73311PDBV, Package_TO_SOT_SMD:SOT-23-5, symbol Regulator_Linear:TLV73311PDBV
- added J10: OLED_2, JumperlessFootprints:Conn_1x4, symbol Connector_Generic:Conn_01x04
- added J9: OLED_1, JumperlessFootprints:Conn_1x4, symbol Connector_Generic:Conn_01x04
- added JP33: Bridge RST, JumperlessFootprints:SolderJumper_2_Open_Small, symbol Jumper:Jumper_2_Small_Open
- added U6: ~, JumperlessFootprints:SolderJumper-Double, symbol JumperlessSymbols:SolderJumperDouble
- R22: value 10K -> 1K
- TP28: symbol Connector:Conn_01x04_Pin -> Connector:Conn_01x08_Pin
Connections:
- net +5V: now also J10.3 (Pin_3), J9.3 (Pin_3)
- net GND: now also J10.4 (Pin_4), J9.4 (Pin_4)
- net GPIO_6: now also TP28.7 (Pin_7), U6.4 (B)
- net GPIO_7: now also TP28.8 (Pin_8), U6.5 (B)
- net I2C_SCL: now also U6.1 (A)
- net I2C_SDA: now also U6.2 (A)
- net at JP7.2 (B), U5.18 (GPIO18): now also JP33.1 (A)
- net at JP8.2 (B), U5.19 (GPIO19): now also JP33.2 (B)
- new net OLED_SCL: J10.2 (Pin_2), J9.2 (Pin_2), U6.6 (C)
- new net OLED_SDA: J10.1 (Pin_1), J9.1 (Pin_1), U6.3 (C)
Other:
- note removed: "So I can swap over to the LDO if this SMPS is being a dick"
- moved on the sheet: JP11, R26, R27
