File: Jumperless23V50/PSRAMmod/PSRAMmod.kicad_sch (KiCad schematic)
At the start: 53 parts, among them J1 NANO_RESET_1, J2 Pogo, U1 APS6404L-3SQRx-ZR, U2 W25Q128JVS

Commit message: Add PSRAM mod files
Parts:
- D1, D10, D11, D12, D13, D14, D15, D16, D17, D18, D19, D2, D20, D21, D22, D23, D24, D25, D26, D27, D28, D29, D3, D30, D31, D32, D33, D34, D35, D36, D37, D38, D39, D4, D40, D41, D42, D43, D5, D6, D7, D8, D9: LCSC (none) -> C5349953
- J2: footprint (none) -> JumperlessFootprints:Pogo_pin_YZP0120-16020-01; LCSC Part (none) -> C5157215
- JP1: footprint (none) -> JumperlessFootprints:SolderJumper-3_P1.3mm_Bridged12_Pad1.0x1.5mm
- TP2: footprint JumperlessFootprints:PINHEADER-1x1_vertical -> (none)
- TP5: footprint JumperlessFootprints:PINHEADER-1x1_vertical -> JumperlessFootprints:TestPoint_D0.75mm
- U1: LCSC Part (none) -> C3040877
- U2: footprint Package_SO:SOIC-8_5.3x5.3mm_P1.27mm -> JumperlessFootprints:SOIC-8_Castillated; LCSC (none) -> C97521; LCSC Part # (none) -> C97521
