File: Jumperless23V50/PSRAMmod/PSRAMmod.kicad_pcb (KiCad board)
At the start: 2 copper layers, 59.1 x 26.1 mm, 58 parts, among them J1 NANO_RESET_1, J14 5V, J2 Pogo, U1 APS6404L-3SQRx-ZR, U2 W25Q128JVS

Commit message: add random stuff
Parts:
- removed A1: Arduino_Nano_v3.x, JumperlessFootprints:Arduino_Nano
- removed J14: 5V, JumperlessFootprints:PINHEADER-1x1_vertical
- removed JP8: Reset 1, JumperlessFootprints:SolderJumper_2_Bridged_Small
- removed REF**: Minimum_CE_Mark, JumperlessFootprints:Minimum_CE_Mark
- removed the TP20 at (156.5, 123.5)
Routing:
- net GND: track 215.3 -> 214.8 mm
- removed copper zone on F.Cu, net (none)
