File: Jumperless23V50/ProbeSenseNumbers/ProbeSenseNumbers.kicad_pcb (KiCad board)
At the start: 2 copper layers, 80.8 x 50.8 mm, 72 parts, among them J3 TopIn, J31 + - top, J32 + - bottom, J34 TopOut, J35 BottomIn, J4 BottomOut

Commit message: mostly screw with releases and actions
Other:
- board text added: "PCB3D_BR_SENSE"
- board text added: "PCB3D_TL_SENSE"
